Commit message: Fix collision and remove vizualisation

File: guidebot_description/urdf/sensors/sweep.gazebo.xacro (robot description, xacro)
@@ -5,5 +5,5 @@
       <sensor type="ray" name="${name}">
         <pose>0 0 0 0 0 0</pose>
-        <visualize>true</visualize>
+        <visualize>false</visualize>
         <update_rate>${update_rate}</update_rate>
         <ray>

File: guidebot_description/urdf/sensors/sweep.urdf.xacro (robot description, xacro)
@@ -24,5 +24,4 @@
     </joint>
     <link name="${name}_link">
-      <!--
       <visual>
         <origin xyz="0 0 -0.033" rpy="0 0 0"/>
@@ -33,9 +32,9 @@
       </visual>
       <collision>
+        <origin xyz="0 0 -0.033" rpy="0 0 0"/>
         <geometry>
           <mesh filename="${mesh}" />
         </geometry>
       </collision>
-      -->
       <inertial>
         <mass value="${mass}" />
