Commit message: Integrate move_base to cartograper test

File: guidebot_description/urdf/base/diff_drive_base.gazebo.xacro (robot description, xacro)
@@ -16,3 +16,22 @@
     </gazebo>
   </macro>
+  <gazebo reference="imu_link">
+   <gravity>true</gravity>
+   <sensor name="imu_sensor" type="imu">
+     <always_on>true</always_on>
+     <update_rate>100</update_rate>
+     <visualize>true</visualize>
+     <topic>__default_topic__</topic>
+     <plugin filename="libgazebo_ros_imu_sensor.so" name="imu_plugin">
+       <topicName>imu</topicName>
+       <bodyName>imu_link</bodyName>
+       <updateRateHZ>10.0</updateRateHZ>
+       <gaussianNoise>0.0</gaussianNoise>
+       <xyzOffset>0 0 0</xyzOffset>
+       <rpyOffset>0 0 0</rpyOffset>
+       <frameName>imu_link</frameName>
+     </plugin>
+     <pose>0 0 0 0 0 0</pose>
+   </sensor>
+ </gazebo>
 </robot>

File: guidebot_description/urdf/base/diff_drive_base.urdf.xacro (robot description, xacro)
@@ -42,8 +42,15 @@
     <!-- Base footprint -->
     <link name="base_footprint"/>
-    <joint name="base_footprint_link" type="fixed">
+    <joint name="base_footprint_joint" type="fixed">
       <origin xyz="0 0 ${wheel_radius}" rpy="0 0 0"/>
       <parent link="base_footprint"/>
       <child link="base_link"/>
+    </joint>
+    <!-- IMU link -->
+    <link name="imu_link"/>
+    <joint name="imu_joint" type="fixed">
+      <origin xyz="0 0 ${wheel_radius}" rpy="0 0 0"/>
+      <parent link="base_footprint"/>
+      <child link="imu_link"/>
     </joint>
     <!-- Macros -->

File: guidebot_description/urdf/wheels/drive_wheel.urdf.xacro (robot description, xacro)
@@ -33,5 +33,5 @@
       <child link="${name}_link"/>
       <axis xyz="0 0 1"/>
-      <limit effort="1" velocity="1"/>
+      <limit effort="1000" velocity="1000"/>
     </joint>
     <!-- Transmission -->
