Commit message: Make base_footprint kinematic

File: guidebot_description/urdf/base/holonomic_base.gazebo.xacro (robot description, xacro)
@@ -6,13 +6,24 @@
     </gazebo>
     <gazebo reference="base_footprint">
-      <kp>100000000.0</kp>
-      <kd>10.0</kd>
-      <mu1>0.1</mu1>
-      <mu2>0.1</mu2>
-      <fdir1>1 0 0</fdir1>
-      <maxVel>10.0</maxVel>
-      <minDepth>0.0005</minDepth>
-      <laserRetro>0</laserRetro>
+      <kinematic>true</kinematic>
     </gazebo>
   </macro>
+  <gazebo>
+    <plugin name="object_controller" filename="libgazebo_ros_planar_move.so">
+      <commandTopic>cmd_vel</commandTopic>
+      <odometryTopic>/odom</odometryTopic>
+      <odometryFrame>odom</odometryFrame>
+      <odometryRate>20.0</odometryRate>
+      <robotBaseFrame>base_footprint</robotBaseFrame>
+    </plugin>
+<!--
+    <plugin name="object_controller" filename="libgazebo_ros_force_based_move.so">
+      <commandTopic>cmd_vel</commandTopic>
+      <odometryTopic>/odom</odometryTopic>
+      <odometryFrame>odom</odometryFrame>
+      <odometryRate>20.0</odometryRate>
+      <robotBaseFrame>base_footprint</robotBaseFrame>
+    </plugin>
+ -->
+  </gazebo>
 </robot>

File: guidebot_description/urdf/base/holonomic_base.urdf.xacro (robot description, xacro)
@@ -7,5 +7,5 @@
   <property name="M_PI" value="3.1415926535897931"/>
   <!-- Base footprint offset -->
-  <property name="base_footprint_height_offset" value="0.190"/>
+  <property name="base_footprint_height_offset" value="0.19"/> <!-- old value 0.19 -->
   <!-- Inertia -->
   <macro name="cylinder_inertia" params="m r h">
@@ -35,11 +35,26 @@
       <!-- TODO: update according to real base properties -->
       <inertial>
+        <mass value="10.0" />
+        <origin xyz="0 0 0" />
+        <cylinder_inertia m="10.0" r="0.3" h="0.2" />
+      </inertial>
+    <!--
+      <inertial>
         <origin xyz="-0.00000106 0.00000109 0.0000387" rpy="0 0 0"/>
         <mass value="15.0"/>
         <inertia ixx="0.465408937" ixy="0.002160024" ixz="-0.001760255" iyy="0.483193291" iyz="-0.000655952" izz="0.550939703"/>
       </inertial>
+   -->
     </link>
     <!-- Base footprint -->
-    <link name="base_footprint"/>
+    <link name="base_footprint">
+      <collision>
+        <origin xyz="0 0 0" rpy="0 0 0"/>
+        <geometry>
+          <cylinder length="0.01" radius="0.3"/>
+        </geometry>
+        <material name="orange"/>
+      </collision>
+    </link>
     <joint name="base_footprint_joint" type="fixed">
       <origin xyz="0 0 ${base_footprint_height_offset}" rpy="0 0 0"/>

File: guidebot_description/urdf/wheels/diff_drive/drive_wheel.gazebo.xacro (robot description, xacro)
@@ -3,7 +3,12 @@
   <macro name="drive_wheel_gazebo" params="name">
     <!-- Contact model for the wheel surface -->
+    <!-- TEMPORARY: Set friction very low and control base with gazebo planar move -->
    <gazebo reference="${name}_link">
-     <kp>1000000.0</kp>
+     <!--
+     <kp>100000.0</kp>
      <kd>100.0</kd>
+      -->
+     <kp>0.1</kp>
+     <kd>0.1</kd>
      <mu1>1.0</mu1>
      <mu2>1.0</mu2>

File: guidebot_description/urdf/wheels/holonomic/wheel_assembly.gazebo.xacro (robot description, xacro)
@@ -16,6 +16,6 @@
     <gazebo reference="${name}">
       <material>Gazebo/${color}</material>
-      <kp>100000.0</kp>
-      <kd>10.0</kd>
+      <kp>1000000.0</kp>
+      <kd>100.0</kd>
       <mu1>1</mu1>
       <mu2>1</mu2>

File: guidebot_description/urdf/wheels/holonomic/wheel_assembly.urdf.xacro (robot description, xacro)
@@ -42,7 +42,9 @@
       </visual>
       <collision>
+        <!--
         <geometry>
           <cylinder length="${wheel_width}" radius="${wheel_radius}"/>
         </geometry>
+         -->
       </collision>
     </link>
