Commit message: Add working Scanse sweep simulated scanner

File: guidebot_description/robots/diff_drive.xacro (robot description, xacro)
@@ -5,5 +5,12 @@
   <!-- Set up definitions of parts of robot body -->
   <include filename="../urdf/base/diff_drive_base.urdf.xacro"/>
+  <include filename="../urdf/sensors/sweep.urdf.xacro"/>
   <!-- Use macros to define the actual robot -->
-  <xacro:base/>
+  <base/>
+  <joint name="sweep_mount_joint" type="fixed">
+    <origin xyz="0 0 0.142" rpy="0 0 0"/>
+    <parent link="base_link"/>
+    <child link="sweep_mount_link"/>
+  </joint>
+  <sweep name="sweep" ros_topic="scan" min_angle="${-pi}" max_angle="${pi}"/>
 </robot>

Commit message: Make makro for gazebo urdf

File: guidebot_description/robots/diff_drive.xacro (robot description, xacro)
@@ -6,4 +6,5 @@
   <include filename="../urdf/base/diff_drive_base.urdf.xacro"/>
   <include filename="../urdf/sensors/sweep.urdf.xacro"/>
+  <include filename="../urdf/sensors/imu.urdf.xacro"/>
   <!-- Use macros to define the actual robot -->
   <base/>
@@ -14,3 +15,4 @@
   </joint>
   <sweep name="sweep" ros_topic="scan" min_angle="${-pi}" max_angle="${pi}"/>
+  <imu/>
 </robot>

File: guidebot_description/urdf/base/diff_drive_base.gazebo.xacro (robot description, xacro)
@@ -16,22 +16,3 @@
     </gazebo>
   </macro>
-  <gazebo reference="imu_link">
-   <gravity>true</gravity>
-   <sensor name="imu_sensor" type="imu">
-     <always_on>true</always_on>
-     <update_rate>100</update_rate>
-     <visualize>true</visualize>
-     <topic>__default_topic__</topic>
-     <plugin filename="libgazebo_ros_imu_sensor.so" name="imu_plugin">
-       <topicName>imu</topicName>
-       <bodyName>imu_link</bodyName>
-       <updateRateHZ>10.0</updateRateHZ>
-       <gaussianNoise>0.0</gaussianNoise>
-       <xyzOffset>0 0 0</xyzOffset>
-       <rpyOffset>0 0 0</rpyOffset>
-       <frameName>imu_link</frameName>
-     </plugin>
-     <pose>0 0 0 0 0 0</pose>
-   </sensor>
- </gazebo>
 </robot>

File: guidebot_description/urdf/base/diff_drive_base.urdf.xacro (robot description, xacro)
@@ -1,5 +1,5 @@
 <?xml version="1.0"?>
 <!-- Guidebot differential drive base -->
-<robot xmlns:xacro="http://www.ros.org/wiki/xacro">
+<robot xmlns:xacro="http://ros.org/wiki/xacro">
   <include filename="diff_drive_base.gazebo.xacro"/>
   <include filename="../wheels/drive_wheel.urdf.xacro"/>
@@ -47,11 +47,4 @@
       <child link="base_link"/>
     </joint>
-    <!-- IMU link -->
-    <link name="imu_link"/>
-    <joint name="imu_joint" type="fixed">
-      <origin xyz="0 0 ${wheel_radius}" rpy="0 0 0"/>
-      <parent link="base_footprint"/>
-      <child link="imu_link"/>
-    </joint>
     <!-- Macros -->
     <drive_wheel name="wheel_right" radius="${wheel_radius}" width="${wheel_width}" separation="${wheel_separation}" reflect="1.0" parent="base_link"/>

File: guidebot_description/urdf/plugins.gazebo.xacro (robot description, xacro)
@@ -1,4 +1,4 @@
 <?xml version="1.0"?>
-<robot xmlns:xacro="http://www.ros.org/wiki/xacro">
+<robot xmlns:xacro="http://ros.org/wiki/xacro">
   <gazebo>
     <plugin name="gazebo_ros_control" filename="libgazebo_ros_control.so">
