Commit message: Add exploration rapp

File: guidebot_description/urdf/wheels/drive_wheel.urdf.xacro (robot description, xacro)
@@ -33,5 +33,5 @@
       <child link="${name}_link"/>
       <axis xyz="0 0 1"/>
-      <limit effort="1000" velocity="1000"/>
+      <limit effort="10000" velocity="10000"/>
     </joint>
     <!-- Transmission -->
